Commit message: add IMU and camera info for H2

File: robots/h2_description/H2.urdf (robot description, URDF)
Before this commit: robot H2, 34 links, 33 joints
Links:
- added link camera
- added link imu_in_pelvis
- added link imu_in_torso
Joints:
- added joint camera: type fixed, parent head_yaw_link, child camera, origin xyz=0.08667 0.03 0.0099 rpy=0 0 0
- added joint imu_in_pelvis_joint: type fixed, parent pelvis, child imu_in_pelvis, origin xyz=-0.055 0 -0.0589 rpy=0 0 0
- added joint imu_in_torso_joint: type fixed, parent torso_link, child imu_in_torso, origin xyz=-0.06382 -0.06538 0.29588 rpy=0 0 0

File: robots/h2_description/H2_dae.urdf (robot description, URDF)
Before this commit: robot H2, 34 links, 33 joints
Links:
- added link camera
- added link imu_in_pelvis
- added link imu_in_torso
Joints:
- added joint camera: type fixed, parent head_yaw_link, child camera, origin xyz=0.08667 0.03 0.0099 rpy=0 0 0
- added joint imu_in_pelvis_joint: type fixed, parent pelvis, child imu_in_pelvis, origin xyz=-0.055 0 -0.0589 rpy=0 0 0
- added joint imu_in_torso_joint: type fixed, parent torso_link, child imu_in_torso, origin xyz=-0.06382 -0.06538 0.29588 rpy=0 0 0
