Commit message: update b2 urdf

File: robots/b2_description/urdf/b2_description.urdf (robot description, URDF)
Before this commit: robot b2_description, 37 links, 36 joints
Links:
- link FL_thigh: geometry collision box size=0.25 0.028 0.04; visual mesh filename=package://b2_description/meshes/FL_thigh.dae
