Commit message: update r1_{a5,a7} arm joints max velocity

File: robots/r1_a5_description/r1_a5.urdf (robot description, URDF)
Before this commit: robot A5, 14 links, 13 joints
Joints:
- joint head_pitch_joint: limit lower=-0.62832 upper=0.62832 effort=33 velocity=52.4 -> lower=-0.62832 upper=0.62832 effort=33 velocity=33.4
- joint left_elbow_joint: limit lower=-0.97564 upper=2.1852 effort=33 velocity=52.4 -> lower=-0.97564 upper=2.1852 effort=33 velocity=33.4
- joint left_shoulder_yaw_joint: limit lower=-1.9199 upper=1.9199 effort=33 velocity=52.4 -> lower=-1.9199 upper=1.9199 effort=33 velocity=33.4
- joint left_wrist_roll_joint: limit lower=-1.9199 upper=1.9199 effort=33 velocity=52.4 -> lower=-1.9199 upper=1.9199 effort=33 velocity=33.4
- joint right_elbow_joint: limit lower=-0.97564 upper=2.1852 effort=33 velocity=52.4 -> lower=-0.97564 upper=2.1852 effort=33 velocity=33.4
- joint right_shoulder_yaw_joint: limit lower=-1.9199 upper=1.9199 effort=33 velocity=52.4 -> lower=-1.9199 upper=1.9199 effort=33 velocity=33.4
- joint right_wrist_roll_joint: limit lower=-1.9199 upper=1.9199 effort=33 velocity=52.4 -> lower=-1.9199 upper=1.9199 effort=33 velocity=33.4

File: robots/r1_a7_description/r1_a7.urdf (robot description, URDF)
Before this commit: robot A7, 18 links, 17 joints
Joints:
- joint head_pitch_joint: limit lower=-0.62832 upper=0.62832 effort=33 velocity=52.4 -> lower=-0.62832 upper=0.62832 effort=33 velocity=33.4
- joint left_elbow_joint: limit lower=-0.97564 upper=2.1852 effort=33 velocity=52.4 -> lower=-0.97564 upper=2.1852 effort=33 velocity=33.4
- joint left_shoulder_yaw_joint: limit lower=-1.9199 upper=1.9199 effort=33 velocity=52.4 -> lower=-1.9199 upper=1.9199 effort=33 velocity=33.4
- joint left_wrist_roll_joint: limit lower=-1.9199 upper=1.9199 effort=33 velocity=52.4 -> lower=-1.9199 upper=1.9199 effort=33 velocity=33.4
- joint right_elbow_joint: limit lower=-0.97564 upper=2.1852 effort=33 velocity=52.4 -> lower=-0.97564 upper=2.1852 effort=33 velocity=33.4
- joint right_shoulder_yaw_joint: limit lower=-1.9199 upper=1.9199 effort=33 velocity=52.4 -> lower=-1.9199 upper=1.9199 effort=33 velocity=33.4
- joint right_wrist_roll_joint: limit lower=-1.9199 upper=1.9199 effort=33 velocity=52.4 -> lower=-1.9199 upper=1.9199 effort=33 velocity=33.4
